Commit message: update params

File: isaac_ros-dev/src/go2_description/urdf/go2_nav2_nvblox.urdf (robot description, URDF)
Before this commit: robot go2, 32 links, 31 joints
Joints:
- joint laser_joint: origin xyz=0.22 0 0.12 rpy=0 0 0 -> xyz=0 0 0.17 rpy=0 0 0

Commit message: Added isaac_ros_map_localization as a submodule

File: isaac_ros-dev/src/go2_description/urdf/go2_nav2_nvblox.urdf (robot description, URDF)
Before this commit: robot go2, 32 links, 31 joints
Links:
- link laser: geometry collision cylinder length=0.05 radius=0.035; visual cylinder length=0.055 radius=0.035
Joints:
- joint laser_joint: origin xyz=0 0 0.17 rpy=0 0 0 -> xyz=0 0 0.27 rpy=0 0 0

Commit message: updated repo to include zedxmini integration

File: isaac_ros-dev/src/go2_description/urdf/go2_nav2_nvblox.urdf (robot description, URDF)
Before this commit: robot go2, 32 links, 31 joints
Joints:
- added joint zed_joint: type fixed, parent base_link, child zed_camera_link, origin xyz=0.19 0.0 0.20 rpy=0 0 0

Commit message: Latest update working with OWL-nano and zed camera

File: isaac_ros-dev/src/go2_description/urdf/go2_nav2_nvblox.urdf (robot description, URDF)
Before this commit: robot go2, 32 links, 32 joints
Joints:
- removed joint zed_joint
