Commit message: update for amigo

File: src/go2_description/urdf/go2.urdf.xacro (robot description, xacro)
@@ -1258,4 +1258,116 @@
       xyz="0 0 0" />
   </joint>
+  <link
+    name="gps">
+    <inertial>
+      <origin
+        xyz="0 0 0"
+        rpy="0 0 0" />
+      <mass
+        value="0" />
+      <inertia
+        ixx="0"
+        ixy="0"
+        ixz="0"
+        iyy="0"
+        iyz="0"
+        izz="0" />
+    </inertial>
+  </link>
+  <joint
+    name="gps_joint"
+    type="fixed">
+    <origin
+      xyz="0.290 0 0.155"
+      rpy="0 0 0" />
+    <parent
+      link="base_link" />
+    <child
+      link="gps" />
+    <axis
+      xyz="0 0 0" />
+  </joint>
+  <link name="laser">
+    <visual>
+      <origin xyz="0 0 0" rpy="0 0 0" />
+      <geometry>
+        <cylinder radius="0.035" length="0.055" />
+      </geometry>
+      <material name="">
+        <color rgba="1 1 1 1" />
+      </material>
+    </visual>
+    <collision>
+      <origin xyz="0 0 0" rpy="0 0 0" />
+      <geometry>
+        <cylinder radius="0.035" length="0.05" />
+      </geometry>
+    </collision>
+  </link>
+  <joint name="laser_joint" type="fixed">
+    <parent link="base_link"/>
+    <child link="laser"/>
+    <origin xyz="0 0 0.27" rpy="0 0 3.14"/>
+  </joint>
+    <!-- <link
+    name="bno055">
+    <inertial>
+      <origin
+        xyz="0 0 0"
+        rpy="0 0 0" />
+      <mass
+        value="0" />
+      <inertia
+        ixx="0"
+        ixy="0"
+        ixz="0"
+        iyy="0"
+        iyz="0"
+        izz="0" />
+    </inertial>
+  </link>
+  <joint
+    name="bno055_imu_joint"
+    type="fixed">
+    <origin
+      xyz="0.200 0.00 0.060"
+      rpy="0 0 0" />
+    <parent
+      link="base_link" />
+    <child
+      link="bno055" />
+    <axis
+      xyz="0 0 0" />
+  </joint> -->
+  <!-- <link
+    name="velodyne">
+    <inertial>
+      <origin
+        xyz="0 0 0"
+        rpy="0 0 0" />
+      <mass
+        value="0" />
+      <inertia
+        ixx="0"
+        ixy="0"
+        ixz="0"
+        iyy="0"
+        iyz="0"
+        izz="0" />
+    </inertial>
+  </link>
+  <joint
+    name="velodyne_joint"
+    type="fixed">
+    <origin
+      xyz="-0.02 0.0 0.26"
+      rpy="0 0 0" />
+    <parent
+      link="base_link" />
+    <child
+      link="velodyne" />
+    <axis
+      xyz="0 0 0" />
+  </joint> -->
   <xacro:include
           filename="$(find zed_wrapper)/urdf/zed_macro.urdf.xacro"/>

Commit message: chore: update Jetson Thor AGX bringup

File: src/go2_description/urdf/go2.urdf.xacro (robot description, xacro)
@@ -1,7 +1,8 @@
 <?xml version="1.0" encoding="utf-8"?>
 <robot name="go2" xmlns:xacro="http://www.ros.org/wiki/xacro">
-  <xacro:arg name="camera_name"   default="zed"/>
-  <xacro:arg name="camera_model"  default="zedxm"/>   <!-- zed, zed2i, zedm, zedx, zedxm … -->
-  <xacro:arg name="use_zed_localization" default="false"/>
+  <xacro:arg name="camera_name" default="camera"/>
+  <xacro:arg name="camera_model" default="d455"/>
+  <xacro:arg name="camera_xyz" default="0.350 0.000 0.200"/>
+  <xacro:arg name="camera_rpy" default="0.000 0.000 0.000"/>
   <link
     name="base_link">
@@ -1370,26 +1371,83 @@
       xyz="0 0 0" />
   </joint> -->
-  <xacro:include
-          filename="$(find zed_wrapper)/urdf/zed_macro.urdf.xacro"/>
-  <xacro:zed_camera name="zed"
-                    model="zedxm">
-    <!-- block required by the macro, but we don’t need it -->
-    <gnss_origin/>
-  </xacro:zed_camera>
-  <!-- ZED publishes TF -> base_link (we don't use this) -->
-  <xacro:if value="$(arg use_zed_localization)">
-    <joint name="zed_mount" type="fixed">
-      <parent link="zed_camera_link"/>
-      <child  link="base_link"/>
-      <origin xyz="0.32 0.0 0.0725" rpy="0 0 0"/>
+  <xacro:macro name="realsense_stream_frames" params="name stream parent xyz">
+    <link name="${name}_${stream}_frame"/>
+    <joint name="${name}_${stream}_joint" type="fixed">
+      <parent link="${parent}"/>
+      <child link="${name}_${stream}_frame"/>
+      <origin xyz="${xyz}" rpy="0 0 0"/>
     </joint>
-  </xacro:if>
-  <!-- EKF publishes odom, camera is child of base_link -->
-  <xacro:unless value="$(arg use_zed_localization)">
-    <joint name="zed_mount" type="fixed">
+    <link name="${name}_${stream}_optical_frame"/>
+    <joint name="${name}_${stream}_optical_joint" type="fixed">
+      <parent link="${name}_${stream}_frame"/>
+      <child link="${name}_${stream}_optical_frame"/>
+      <origin xyz="0 0 0" rpy="-1.57079632679 0 -1.57079632679"/>
+    </joint>
+  </xacro:macro>
+  <xacro:macro name="realsense_imu_frames" params="name parent">
+    <link name="${name}_accel_frame"/>
+    <joint name="${name}_accel_joint" type="fixed">
+      <parent link="${parent}"/>
+      <child link="${name}_accel_frame"/>
+      <origin xyz="0 0 0" rpy="0 0 0"/>
+    </joint>
+    <link name="${name}_accel_optical_frame"/>
+    <joint name="${name}_accel_optical_joint" type="fixed">
+      <parent link="${name}_accel_frame"/>
+      <child link="${name}_accel_optical_frame"/>
+      <origin xyz="0 0 0" rpy="-1.57079632679 0 -1.57079632679"/>
+    </joint>
+    <link name="${name}_gyro_frame"/>
+    <joint name="${name}_gyro_joint" type="fixed">
+      <parent link="${parent}"/>
+      <child link="${name}_gyro_frame"/>
+      <origin xyz="0 0 0" rpy="0 0 0"/>
+    </joint>
+    <link name="${name}_gyro_optical_frame"/>
+    <joint name="${name}_gyro_optical_joint" type="fixed">
+      <parent link="${name}_gyro_frame"/>
+      <child link="${name}_gyro_optical_frame"/>
+      <origin xyz="0 0 0" rpy="-1.57079632679 0 -1.57079632679"/>
+    </joint>
+    <link name="${name}_imu_optical_frame"/>
+    <joint name="${name}_imu_optical_joint" type="fixed">
+      <parent link="${name}_gyro_optical_frame"/>
+      <child link="${name}_imu_optical_frame"/>
+      <origin xyz="0 0 0" rpy="0 0 0"/>
+    </joint>
+  </xacro:macro>
+  <xacro:macro name="realsense_camera_frames" params="name xyz rpy">
+    <link name="${name}_link">
+      <visual>
+        <origin xyz="0 0 0" rpy="0 0 0"/>
+        <geometry>
+          <box size="0.090 0.025 0.025"/>
+        </geometry>
+        <material name="camera_color">
+          <color rgba="0.1 0.1 0.1 1"/>
+        </material>
+      </visual>
+      <collision>
+        <origin xyz="0 0 0" rpy="0 0 0"/>
+        <geometry>
+          <box size="0.090 0.025 0.025"/>
+        </geometry>
+      </collision>
+    </link>
+    <joint name="${name}_joint" type="fixed">
       <parent link="base_link"/>
-      <child  link="zed_camera_link"/>
-      <origin xyz="0.32 0.0 0.0725" rpy="0 0 0"/>
+      <child link="${name}_link"/>
+      <origin xyz="${xyz}" rpy="${rpy}"/>
     </joint>
-  </xacro:unless>
+    <xacro:realsense_stream_frames name="${name}" stream="depth" parent="${name}_link" xyz="0 0 0"/>
+    <xacro:realsense_stream_frames name="${name}" stream="color" parent="${name}_link" xyz="0 0 0"/>
+    <!-- D455 IR imagers: infra1 is left, infra2 is right. Values are meters. -->
+    <xacro:realsense_stream_frames name="${name}" stream="infra1" parent="${name}_link" xyz="0.36 0.05 0.20"/>
+    <xacro:realsense_stream_frames name="${name}" stream="infra2" parent="${name}_link" xyz="0.36 -0.05 0.20"/>
+    <xacro:realsense_imu_frames name="${name}" parent="${name}_link"/>
+  </xacro:macro>
+  <xacro:realsense_camera_frames
+    name="$(arg camera_name)"
+    xyz="$(arg camera_xyz)"
+    rpy="$(arg camera_rpy)"/>
 </robot>

Commit message: Add RealSense YOLOv8 follow workflow

File: src/go2_description/urdf/go2.urdf.xacro (robot description, xacro)
@@ -3,6 +3,16 @@
   <xacro:arg name="camera_name" default="camera"/>
   <xacro:arg name="camera_model" default="d455"/>
-  <xacro:arg name="camera_xyz" default="0.350 0.000 0.200"/>
+  <xacro:arg name="camera_xyz" default="0.340 0.000 0.200"/>
   <xacro:arg name="camera_rpy" default="0.000 0.000 0.000"/>
+  <xacro:arg name="camera_rig_enable" default="false"/>
+  <xacro:arg name="camera0_xyz" default="0.340 0.000 0.200"/>
+  <xacro:arg name="camera0_rpy" default="0.000 0.000 0.000"/>
+  <xacro:arg name="camera1_xyz" default="0.265 0.0601 0.200"/>
+  <xacro:arg name="camera1_rpy" default="0.000 0.000 1.57079632679"/>
+  <xacro:arg name="camera2_xyz" default="0.265 -0.0601 0.200"/>
+  <xacro:arg name="camera2_rpy" default="0.000 0.000 -1.57079632679"/>
+  <xacro:property name="d455_ir_left_y" value="0.050"/>
+  <xacro:property name="d455_ir_right_y" value="-0.050"/>
+  <xacro:property name="d455_color_y" value="-0.012"/>
   <link
     name="base_link">
@@ -1440,14 +1450,30 @@
       <origin xyz="${xyz}" rpy="${rpy}"/>
     </joint>
-    <xacro:realsense_stream_frames name="${name}" stream="depth" parent="${name}_link" xyz="0 0 0"/>
-    <xacro:realsense_stream_frames name="${name}" stream="color" parent="${name}_link" xyz="0 0 0"/>
-    <!-- D455 IR imagers: infra1 is left, infra2 is right. Values are meters. -->
-    <xacro:realsense_stream_frames name="${name}" stream="infra1" parent="${name}_link" xyz="0.36 0.05 0.20"/>
-    <xacro:realsense_stream_frames name="${name}" stream="infra2" parent="${name}_link" xyz="0.36 -0.05 0.20"/>
+    <!-- D455 camera_link is modeled at the stereo center. Infra/depth offsets are local to that link. -->
+    <xacro:realsense_stream_frames name="${name}" stream="depth" parent="${name}_link" xyz="0 ${d455_ir_left_y} 0"/>
+    <xacro:realsense_stream_frames name="${name}" stream="color" parent="${name}_link" xyz="0 ${d455_color_y} 0"/>
+    <xacro:realsense_stream_frames name="${name}" stream="infra1" parent="${name}_link" xyz="0 ${d455_ir_left_y} 0"/>
+    <xacro:realsense_stream_frames name="${name}" stream="infra2" parent="${name}_link" xyz="0 ${d455_ir_right_y} 0"/>
     <xacro:realsense_imu_frames name="${name}" parent="${name}_link"/>
   </xacro:macro>
-  <xacro:realsense_camera_frames
-    name="$(arg camera_name)"
-    xyz="$(arg camera_xyz)"
-    rpy="$(arg camera_rpy)"/>
+  <xacro:if value="$(arg camera_rig_enable)">
+    <xacro:realsense_camera_frames
+      name="camera0"
+      xyz="$(arg camera0_xyz)"
+      rpy="$(arg camera0_rpy)"/>
+    <xacro:realsense_camera_frames
+      name="camera1"
+      xyz="$(arg camera1_xyz)"
+      rpy="$(arg camera1_rpy)"/>
+    <xacro:realsense_camera_frames
+      name="camera2"
+      xyz="$(arg camera2_xyz)"
+      rpy="$(arg camera2_rpy)"/>
+  </xacro:if>
+  <xacro:unless value="$(arg camera_rig_enable)">
+    <xacro:realsense_camera_frames
+      name="$(arg camera_name)"
+      xyz="$(arg camera_xyz)"
+      rpy="$(arg camera_rpy)"/>
+  </xacro:unless>
 </robot>
