Commit message: Add explore + deliver-swag behaviors and go2_arm package; prune stale maps
Behaviors / nodes (go2_control):
- New "explore the area" (manual-drive mapping + ArUco record/save) and
  "deliver swag" (Nav2 staging + ArUco visual-servo + CubeMars arm) flows.
- New nodes: aruco_detector_node, aruco_map_store, map_marker_recorder_node,
  deliver_swag_action_server, delivery_geometry, localize_baseline_core,
  plus unit tests for aruco map store, baseline sampling, delivery geometry
  and explore/deliver core.
- Leak localization: costmap perpendicular-baseline sampling + Sit/RiseSit
  recovery.
- Mission supervisor + voice command refactor.

New package:
- go2_arm: gs_usb CubeMars AK45 record/replay (ak45_motor, arm_record_node,
  arm_replay_node, arm_trajectory + test).

Interfaces:
- DeliverSwag.action, PlayArmScript.srv, SaveExploreMap.srv.

Launch / config:
- mapping.launch split + behavior/nav/audio/base updates; nav2 MPPI, EKF,
  and nvblox rviz tuning; removed unused zedxm_rtabmap.launch.py.

Submodules (committed + pushed to forks):
- add unitree_ros2; odas_ros (tunable leak-classifier params); zed-ros2-wrapper
  (package:// mesh URIs); bump zed-ros2-examples and robot_localization.

Autostart / docs:
- setup_robot.sh, amigo.service, amigo_autostart.sh; docs/AGENT_PROMPTS.md,
  docs/EXPLORE_DELIVER_SWAG.md, leak-localization reference paper.

Cleanup:
- Remove stale maps/ and mission_log.txt; gitignore sdk/ and bench scratch.

Co-Authored-By: Claude Opus 4.8 (1M context) <noreply@anthropic.com>

File: src/go2_description/urdf/go2.urdf.xacro (robot description, xacro)
@@ -2,5 +2,5 @@
 <robot name="go2" xmlns:xacro="http://www.ros.org/wiki/xacro">
   <xacro:arg name="camera_name"   default="zed"/>
-  <xacro:arg name="camera_model"  default="zedxm"/>   <!-- zed, zed2i, zedm, zedx, zedxm … -->
+  <xacro:arg name="camera_model"  default="zed2i"/>   <!-- zed, zed2i, zedm, zedx, zedxm … -->
   <xacro:arg name="use_zed_localization" default="false"/>
   <link
@@ -41,17 +41,10 @@
     </collision>
   </link>
-  <joint name="base_footprint_joint" type="fixed">
-    <parent link="base_footprint"/>
-    <child link="base_link"/>
-    <origin xyz="0 0 0" rpy="0 0 0"/>
-  </joint>
-  <link name="base_footprint">
-    <collision>
-      <origin rpy="0 0 0" xyz="0 0 0" />
-      <geometry>
-        <box size="0.3762 0.0935 0.114" />
-      </geometry>
-    </collision>
-    </link>
+  <!-- base_footprint -> base_link is intentionally NOT declared here. It is
+       published dynamically by the base_to_base_tf node (carrying body z + roll/pitch).
+       Declaring it as a fixed URDF joint made robot_state_publisher ALSO broadcast it
+       on /tf_static (identity, no tilt), duplicating/contradicting the dynamic edge.
+       base_link is therefore the URDF root; odom->base_footprint (EKF) and
+       base_footprint->base_link (base_to_base_tf) come from /tf at runtime. -->
   <link
     name="Head_upper">
@@ -1373,5 +1366,5 @@
           filename="$(find zed_wrapper)/urdf/zed_macro.urdf.xacro"/>
   <xacro:zed_camera name="zed"
-                    model="zedxm">
+                    model="$(arg camera_model)">
     <!-- block required by the macro, but we don’t need it -->
     <gnss_origin/>
